File: pcb/micromouse-pcb.kicad_sch (KiCad schematic)
At the start: 40 parts, among them J1_MotorEncoder1 Conn_01x06, J2_MotorEncoder1 Conn_01x06, J3 Conn_01x08, J4 Conn_01x08, Q1 BS170, Q2 TEFT4300, Q3 BS170, Q4 TEFT4300, Q5 BS170, Q6 TEFT4300, Q7 BS170, Q8 TEFT4300, SW1 SW_SPDT, U0 Teensy 4.1, U2 L7805

Commit message: edited pcb
Parts:
- D0: footprint LED_THT:LED_D5.0mm_Clear -> LED_THT:LED_D5.0mm_Horizontal_O1.27mm_Z3.0mm_IRBlack
- D1, D2, D3, D4: footprint SFH_4545:DIO_SFH_4545 -> LED_THT:LED_D5.0mm_Horizontal_O1.27mm_Z3.0mm_IRBlack
- U2: footprint Package_TO_SOT_SMD:TO-252-3_TabPin2 -> Package_TO_SOT_THT:TO-220-3_Vertical
Changed lines of the file:
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@@
 			)
 		)
-		(property "Footprint" "LED_THT:LED_D5.0mm_Clear"
+		(property "Footprint" "LED_THT:LED_D5.0mm_Horizontal_O1.27mm_Z3.0mm_IRBlack"
 			(at 370.84 74.93 0)
 			(effects
@@
 			)
 		)
-		(property "Footprint" "SFH_4545:DIO_SFH_4545"
+		(property "Footprint" "LED_THT:LED_D5.0mm_Horizontal_O1.27mm_Z3.0mm_IRBlack"
 			(at 251.46 118.11 0)
 			(effects
@@
 	)
 	(symbol
+		(lib_id "Regulator_Linear:L7805")
+		(at 346.71 46.99 0)
+		(unit 1)
+		(exclude_from_sim no)
+		(in_bom yes)
+		(on_board yes)
+		(dnp no)
+		(fields_autoplaced yes)
+		(property "Reference" "U2"
+			(at 346.71 40.64 0)
+			(effects
+				(font
+					(size 1.27 1.27)
+				)
+			)
+		)
+		(property "Value" "L7805"
+			(at 346.71 43.18 0)
+			(effects
+				(font
+					(size 1.27 1.27)
+				)
+			)
+		)
+		(property "Footprint" "Package_TO_SOT_THT:TO-220-3_Vertical"
+			(at 347.345 50.8 0)
+			(effects
+				(font
+					(size 1.27 1.27)
+					(italic yes)
+				)
+				(justify left)
+				(hide yes)
+			)
+		)
+		(property "Datasheet" "http://www.st.com/content/ccc/resource/technical/document/datasheet/41/4f/b3/b0/12/d4/47/88/CD00000444.pdf/files/CD00000444.pdf/jcr:content/translations/en.CD00000444.pdf"
+			(at 346.71 48.26 0)
+			(effects
+				(font
+					(size 1.27 1.27)
+				)
+				(hide yes)
+			)
+		)
+		(property "Description" "Positive 1.5A 35V Linear Regulator, Fixed Output 5V, TO-220/TO-263/TO-252"
+			(at 346.71 46.99 0)
+			(effects
+				(font
+					(size 1.27 1.27)
+				)
+				(hide yes)
+			)
+		)
+		(pin "1"
+		)
+		(pin "2"
+		)
+		(pin "3"
+		)
+		(instances
+			(project ""
+				(path "/6bab3514-b9e6-4652-bd2e-edc57bdbde3d"
+					(reference "U2")
+					(unit 1)
+				)
+			)
+		)
+	)
+	(symbol
 		(lib_id "SFH_4545:SFH_4545")
 		(at 332.74 118.11 0)
@@
 			)
 		)
-		(property "Footprint" "SFH_4545:DIO_SFH_4545"
+		(property "Footprint" "LED_THT:LED_D5.0mm_Horizontal_O1.27mm_Z3.0mm_IRBlack"
 			(at 332.74 118.11 0)
 			(effects
@@
 			)
 		)
-		(property "Footprint" "SFH_4545:DIO_SFH_4545"
+		(property "Footprint" "LED_THT:LED_D5.0mm_Horizontal_O1.27mm_Z3.0mm_IRBlack"
 			(at 251.46 176.53 0)
 			(effects
@@
 			)
 		)
-		(property "Footprint" "SFH_4545:DIO_SFH_4545"
+		(property "Footprint" "LED_THT:LED_D5.0mm_Horizontal_O1.27mm_Z3.0mm_IRBlack"
 			(at 334.01 175.26 0)
 			(effects
@@
 					(unit 1)
 				)
-			)
-		)
-	)
-	(symbol
-		(lib_id "Regulator_Linear:L7805")
-		(at 346.71 46.99 0)
-		(unit 1)
-		(exclude_from_sim no)
-		(in_bom yes)
-		(on_board yes)
-		(dnp no)
-		(fields_autoplaced yes)
-		(property "Reference" "U2"
-			(at 346.71 40.64 0)
-			(effects
-				(font
-					(size 1.27 1.27)
-				)
-			)
-		)
-		(property "Value" "L7805"
-			(at 346.71 43.18 0)
-			(effects
-				(font
-					(size 1.27 1.27)
-				)
-			)
-		)
-		(property "Footprint" "Package_TO_SOT_SMD:TO-252-3_TabPin2"
-			(at 347.345 50.8 0)
-			(effects
-				(font
-					(size 1.27 1.27)
-					(italic yes)
-				)
-				(justify left)
-				(hide yes)
-			)
-		)
-		(property "Datasheet" "http://www.st.com/content/ccc/resource/technical/document/datasheet/41/4f/b3/b0/12/d4/47/88/CD00000444.pdf/files/CD00000444.pdf/jcr:content/translations/en.CD00000444.pdf"
-			(at 346.71 48.26 0)
-			(effects
-				(font
-					(size 1.27 1.27)
-				)
-				(hide yes)
-			)
-		)
-		(property "Description" "Positive 1.5A 35V Linear Regulator, Fixed Output 5V, TO-220/TO-263/TO-252"
-			(at 346.71 46.99 0)
-			(effects
-				(font
-					(size 1.27 1.27)
-				)
-				(hide yes)
-			)
-		)
-		(pin "1"
-		)
-		(pin "3"
-		)
-		(pin "2"
-		)
-		(instances
-			(project ""
-				(path "/6bab3514-b9e6-4652-bd2e-edc57bdbde3d"
-					(reference "U2")
-					(unit 1)
-				)
