File: pcb/v2/micromouse-pcb.kicad_sch (KiCad schematic)
At the start: 46 parts, among them J1_MotorEncoder1 Conn_01x06, J2_MotorEncoder1 Conn_01x06, J3 Conn_01x08, J4 Conn_01x08, Q1 BS170, Q2 TEFT4300, Q3 BS170, Q4 TEFT4300, Q5 BS170, Q6 TEFT4300, Q7 BS170, Q8 TEFT4300, SW1 SW_SPDT, U0 Teensy 4.1, U2 L7805

Commit message: should be version after design review
Parts:
- removed D0: LED, LED_THT:LED_D5.0mm, symbol Device:LED
- removed R1_750: R_US, Resistor_SMD:R_1206_3216Metric_Pad1.30x1.75mm_HandSolder, symbol Device:R_US
- added D5, D6: LED, LED_THT:LED_D5.0mm, symbol Device:LED
- added R1_1, R1_2: R_US, Resistor_SMD:R_1206_3216Metric_Pad1.30x1.75mm_HandSolder, symbol Device:R_US
Connections:
- net 5V: now also R1_2.1
- net 7.4V: now also SW1.1 (A), D5.2 (A)
- net GND: now also D6.1 (K), R1_1.1
- new net: D5.1 (K), R1_1.2
- new net: D6.2 (A), R1_2.2
Other:
- moved on the sheet: H1

Commit message: Got gyro in
Parts:
- added J1: Conn_01x08, Connector_PinSocket_2.54mm:PinSocket_1x08_P2.54mm_Vertical, symbol Connector_Generic:Conn_01x08
Connections:
- net 3.3V: now also J1.1 (Pin_1)
- net GND: now also J1.2 (Pin_2), J1.7 (Pin_7)
- net PWM M1_A: now also U0.28 (RX7); no longer U0.18 (A4)
- net PWM M1_B: now also U0.29 (TX7); no longer U0.19 (A5)
- net Signal M2_A: now also U0.40 (A16); no longer U0.16 (A2)
- net Signal M2_B: now also U0.41 (A17); no longer U0.17 (A3)
- new net SCL: J1.3 (Pin_3), U0.19 (A5)
- new net SDA: J1.4 (Pin_4), U0.18 (A4)
- no-connect marks 42 -> 43
Other:
- note added: "GYRO"
- note added: "H-Bridge"
- moved on the sheet: D1, D2, D3, D4, H1, H2, H3, H4, H5, H6, J3, J4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

Commit message: Slight changes to schematic
Changed lines of the file:
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@@
 	(symbol
 		(lib_id "power:GND")
-		(at 378.46 46.99 90)
+		(at 378.46 46.99 0)
 		(unit 1)
 		(exclude_from_sim no)
@@
 		(fields_autoplaced yes)
 		(property "Reference" "#PWR03"
-			(at 384.81 46.99 0)
+			(at 378.46 53.34 0)
 			(effects
 				(font
@@
 		)
 		(property "Value" "GND"
-			(at 382.27 46.9899 90)
+			(at 381 48.2599 0)
 			(effects
 				(font
 					(size 1.27 1.27)
 				)
-				(justify right)
+				(justify left)
 			)
 		)
@@
 	(symbol
 		(lib_id "power:GND")
-		(at 314.96 46.99 270)
+		(at 314.96 46.99 0)
 		(unit 1)
 		(exclude_from_sim no)
@@
 		(fields_autoplaced yes)
 		(property "Reference" "#PWR02"
-			(at 308.61 46.99 0)
+			(at 314.96 53.34 0)
 			(effects
 				(font
@@
 		)
 		(property "Value" "GND"
-			(at 311.15 46.9901 90)
+			(at 317.5 48.2599 0)
 			(effects
 				(font
 					(size 1.27 1.27)
 				)
-				(justify right)
+				(justify left)
 			)
 		)
@@
 	(symbol
 		(lib_id "power:GND")
-		(at 311.15 77.47 270)
+		(at 311.15 77.47 0)
 		(unit 1)
 		(exclude_from_sim no)
@@
 		(fields_autoplaced yes)
 		(property "Reference" "#PWR06"
-			(at 304.8 77.47 0)
+			(at 311.15 83.82 0)
 			(effects
 				(font
@@
 		)
 		(property "Value" "GND"
-			(at 309.88 73.66 90)
+			(at 313.69 78.7399 0)
 			(effects
 				(font
 					(size 1.27 1.27)
 				)
+				(justify left)
 			)
 		)
@@
 	(symbol
 		(lib_id "power:GND")
-		(at 384.81 135.89 90)
+		(at 384.81 135.89 0)
 		(unit 1)
 		(exclude_from_sim no)
@@
 		(fields_autoplaced yes)
 		(property "Reference" "#PWR08"
-			(at 391.16 135.89 0)
+			(at 384.81 142.24 0)
 			(effects
 				(font
@@
 		)
 		(property "Value" "GND"
-			(at 388.62 135.8899 90)
+			(at 387.35 137.1599 0)
 			(effects
 				(font
 					(size 1.27 1.27)
 				)
-				(justify right)
+				(justify left)
 			)
 		)
